File: PCBs/InfiniteRecon/InfiniteRecon.kicad_pcb (KiCad board)
At the start: 4 copper layers, 60 x 60 mm, 127 parts, among them J1 USB_C_Receptacle, J2 Conn_01x04_Pin, U1 BQ25185DLHR, U10 SN74LVC1T45DBV, U11 SN74LVC1T45DBV, U2 MAX17048G_T10, U3 TPS62842DGRR, U4 TLV70018, U5 TPS22918TDBVRQ1, U6 TLV70018, U7 ESP32-S3-WROOM-1, U8 TPL5010DDCR, U9 PCMD3180IRTWR

Commit message: More layout
Parts:
- added C44: 0.1uF, PCM_JLCPCB:C_0402, F.Cu at (181.6, 39.0)
- added C45: 0.1uF, PCM_JLCPCB:C_0402, F.Cu at (210.7, 29.0)
- D6: moved to B.Cu
- J1: footprint Connector_USB:USB_C_Receptacle_GCT_USB4110 -> Connector_USB:USB_C_Receptacle_GCT_USB4105-xx-A_16P_TopMnt_Horizontal
- R4: value 600 -> 1K
- moved U8 199.5 mm to (16.8, 15.2), turned to 90 degrees
- moved C21 197.6 mm to (-13.3, -15.0), turned to -60 degrees
- moved C22 194.7 mm to (16.3, 17.8)
- moved R23 186.1 mm to (18.2, 17.8), turned to 180 degrees
- moved S1 171.0 mm to (13.2, 15.8), turned to -90 degrees
- moved S2 162.3 mm to (22.7, 16.5), turned to -126 degrees
- moved D4 146.4 mm to (20.2, 0.40), turned to -15 degrees
- moved R3 122.4 mm to (19.5, 4.25), turned to 162.5 degrees
- moved R2 120.3 mm to (18.6, 7.10), turned to 162.5 degrees
- moved C1 100.4 mm to (209.1, 43.4), turned to -90 degrees
- moved D1 98.8 mm to (50.0, 16.5)
- moved D2 98.3 mm to (50.0, 21.8)
- moved D3 98.0 mm to (50.0, 26.8)
- moved TP_VSOL_EXT1 83.8 mm to (-18.0, -22.0), turned to -150 degrees
- moved R16 67.1 mm to (101.4, 156.3)
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Routing:
- net GND: track 0.00 -> 4.93 mm, vias 0 -> 2
- net Net-(U1-ISET): track 0.00 -> 3.79 mm
- net Net-(U1-ILIM/VSET): track 0.00 -> 2.57 mm
- net Net-(U1-TS/MR): track 0.00 -> 1.20 mm
- net Net-(MK2-DATA): track 0.00 -> 1.13 mm, vias 0 -> 1

Commit message: Layout more or less done. Still missing i2c pullups and need to redo pinout
Parts:
- removed the C4 at (173.1, 30.5)
- removed the R1 at (98.4, 58.2)
- removed the R22 at (186.3, 129.2)
- removed TP_SYS1: TestPoint, TestPoint:TestPoint_Pad_1.5x1.5mm
- added C45: 0.1uF, PCM_JLCPCB:C_0402, B.Cu at (25.9, -13.3)
- added C46: 1uF, PCM_JLCPCB:C_0603, B.Cu at (20.9, -2.79)
- added R17: 10K, Resistor_SMD:R_0603_1608Metric_Pad0.98x0.95mm_HandSolder, B.Cu at (20.1, -14.7)
- R18, R19, R20, R21: moved to B.Cu
- moved C16 249.4 mm to (-11.6, -0.65), turned to 0 degrees
- moved R14 246.3 mm to (-11.5, 0.90)
- moved U6 238.8 mm to (-7.56, -0.15), turned to 180 degrees
- moved C2 233.6 mm to (-4.94, -0.50), turned to 90 degrees
- moved C15 231.5 mm to (-3.81, -0.97), turned to 90 degrees
- moved C13 224.9 mm to (-2.07, -7.26), turned to -150 degrees
- moved R13 223.7 mm to (-5.16, 6.95), turned to 0 degrees
- moved R12 223.1 mm to (-2.82, -8.56), turned to -150 degrees
- moved U4 221.9 mm to (-5.80, -5.80), turned to 30 degrees
- moved C12 221.8 mm to (-3.86, 4.77), turned to 90 degrees
- moved C3 221.6 mm to (-8.25, -4.96), turned to -60 degrees
- moved C11 221.0 mm to (-8.95, -3.98), turned to -60 degrees
- moved C14 218.8 mm to (-5.06, 4.65), turned to 90 degrees
- moved U5 216.3 mm to (-1.30, 6.00), turned to 180 degrees
- moved R20 215.2 mm to (20.9, -13.3), turned to 30 degrees
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- renumbered C9 to C10, C10 to C11, C11 to C12, C12 to C13, C13 to C14, C14 to C15, C15 to C16, C16 to C17, C17 to C18, C18 to C19, C19 to C20, C20 to C21, C21 to C22, C22 to C23, C23 to C24, C24 to C25, C25 to C26, C26 to C27, C27 to C28, C28 to C29, C45 to C3, C29 to C30, C30 to C31, C31 to C32, C32 to C33, C33 to C34, C34 to C35, C35 to C36, C36 to C37, C37 to C38, C38 to C39, C6 to C4, C39 to C40, C40 to C41, C41 to C42, C42 to C43, C43 to C44, C44 to C5, C3 to C6, C5 to C7, C7 to C8, C8 to C9, R2 to R1, R11 to R10, R12 to R11, R13 to R12, R14 to R13, R15 to R14, R16 to R15, R17 to R16, R3 to R2, R23 to R22, R24 to R23, R25 to R24, R26 to R25, R27 to R26, R28 to R27, R29 to R28, R30 to R29, R4 to R3, R31 to R30, R32 to R31, R33 to R32, R34 to R33, R35 to R34, R36 to R35, R37 to R36, R38 to R37, R5 to R4, R6 to R5, R7 to R6, R8 to R7, R9 to R8, R10 to R9
Connections:
- C2 pad 1: 3V3 -> 3V3_SW
- C30 pad 1: 1V8_SW -> 1V8
- C31 pad 1: 1V8_SW -> 1V8
- C32 pad 1: 1V8_SW -> 1V8
- D2 pad 2: Net-(D2-Pad2) -> VSOl
- R18 pad 1: 3V3_SW -> 3V3
- R18 pad 2: Net-(SIM1-DAT1) -> MISO
- R19 pad 1: 3V3_SW -> 3V3
- R19 pad 2: MISO -> MOSI
- R20 pad 1: 3V3_SW -> 3V3
- R20 pad 2: MOSI -> CS
- R21 pad 1: 3V3_SW -> 3V3
- R21 pad 2: CS -> Net-(SIM1-DAT2)
- SIM1 pad 4: 3V3_SW -> 3V3
Routing:
- net GND: track 4.93 -> 9.40 mm
- net Net-(U1-ISET): track 3.79 -> 0.00 mm
- net Net-(U1-ILIM/VSET): track 2.57 -> 0.00 mm
- net Net-(U1-TS/MR): track 1.20 -> 0.00 mm
- net Net-(MK2-DATA): track 1.13 -> 0.15 mm, vias 1 -> 0
