File: PCBs/InfiniteRecon/audio.kicad_sch (KiCad schematic)
At the start: 0 parts

Commit message: Finished Scem for the most part, awake me needs to look it over one more time
Parts:
- added C17, C18, C19, C20, C21, C22, C23, C24, C25, C26, C27: 0.1uF, PCM_JLCPCB:C_0402, symbol PCM_JLCPCB-Capacitors:0402,100nF
- added C28, C29, C32: 1uF, PCM_JLCPCB:C_0603, symbol Device:C_Small
- added C30, C35, C36: 10uF, PCM_JLCPCB:C_0603, symbol Device:C_Small
- added C31, C33, C34, C37: 0.1uF, PCM_JLCPCB:C_0402, symbol Device:C_Small
- added MK1, MK2, MK3, MK4, MK5, MK6, MK7: T5838, T5838:MIC_T5838, symbol T5838:T5838
- added R17, R18, R19, R20, R21, R22, R23: 33, PCM_JLCPCB:R_0402, symbol Device:R_US
- added R24, R25, R26, R27: 33, PCM_JLCPCB:R_0402, symbol Device:R_Small_US
- added U10, U9: SN74LVC1T45DBV, Package_TO_SOT_SMD:SOT-23-6, symbol Logic_LevelTranslator:SN74LVC1T45DBV
- added U8: PCMD3180IRTWR, Package_DFN_QFN:QFN-28_4x4mm_P0.5mm, symbol JLCImport:PCMD3180IRTWR
Connections:
- new net: MK3.1 (DATA), R19.1
- new net: C30.2, C31.1, U8.2 (AREG)
- new net: C29.2, U8.3 (VREF)
- new net: R25.2, U8.9 (PDMCLK2_GPO2)
- new net: MK1.1 (DATA), R17.1
- new net: C34.1, C35.2, U8.24 (DREG)
- new net: MK2.1 (DATA), R18.1
- new net: MK4.1 (DATA), R20.1
- new net: MK6.1 (DATA), R22.1
- new net: C28.2, U8.5 (MICBIAS)
- new net: R26.2, U8.7 (PDMCLK1_GPO1)
- new net: R27.1, U8.13 (PDMCLK4_GPO4)
- new net: C32.2, C33.1
- new net: MK5.1 (DATA), R21.1
- new net: R24.2, U8.11 (PDMCLK3_GPO3)
- new net: MK7.1 (DATA), R23.1
- new net: MK7.4 (WAKE), U9.3 (A)
- new net 1V8: C17.1, C18.1, C19.1, C20.1, C21.1, C22.1, C23.1, C24.1, C25.1, MK1.2 (SELECT), MK1.7 (VDD), MK2.7 (VDD), MK3.2 (SELECT), MK3.7 (VDD), MK4.7 (VDD), MK5.2 (SELECT), MK5.7 (VDD), MK6.7 (VDD), MK7.5 (THSEL), MK7.7 (VDD), U10.1 (VCCA), U10.3 (A), U8.1 (AVDD), U9.1 (VCCA), U9.5 (DIR)
- new net 3V3: C26.1, C27.1, U10.6 (VCCB), U9.6 (VCCB)
- new net 3V3_SW: C36.2, C37.1, U8.14 (SHDNZ), U8.19 (IOVDD)
- new net GND: C17.2, C18.2, C19.2, C20.2, C21.2, C22.2, C23.2, C24.2, C25.2, C26.2, C27.2, C28.1, C29.1, C30.1, C31.2, C32.1, C33.2, C34.2, C35.1, C36.1, C37.2, MK1.3 (GND), MK2.2 (SELECT), MK2.3 (GND), MK3.3 (GND), MK4.2 (SELECT), MK4.3 (GND), MK5.3 (GND), MK6.2 (SELECT), MK6.3 (GND), MK7.2 (SELECT), MK7.3 (GND), U10.2 (GND), U10.5 (DIR), U8.15 (ADDR1_MISO), U8.16 (ADDR0_SCLK), U8.20 (GPIO1), U8.25 (EP), U8.4 (AVSS), U9.2 (GND)
- new net MIC_THSEL: U10.4 (B)
- new net MIC_WAKE: U9.4 (B)
- new net PDM_CLK_1: MK1.6 (CLK), MK2.6 (CLK), R26.1
- new net PDM_CLK_2: MK3.6 (CLK), MK4.6 (CLK), R25.1
- new net PDM_CLK_3: MK5.6 (CLK), MK6.6 (CLK), R24.1
- new net PDM_CLK_4: MK7.6 (CLK), R27.2
- new net PDM_DIN_1: R17.2, R18.2, U8.6 (PDMDIN1_GPI1)
- new net PDM_DIN_2: R19.2, R20.2, U8.8 (PDMDIN2_GPI2)
- new net PDM_DIN_3: R21.2, R22.2, U8.10 (PDMDIN3_GPI3)
- new net PDM_DIN_4: R23.2, U8.12 (PDMDIN4_GPI4)
- new net SCL_SW: U8.17 (SCL_MOSI)
- new net SDA_SW: U8.18 (SDA_SSZ)
- new net TDM_BCLK: U8.22 (BCLK)
- new net TDM_FSYNC: U8.23 (FSYNC)
- new net TDM_SDOUT: U8.21 (SDOUT)
- no-connect marks 0 -> 12
Other:
- note added: "1V8 -> 3V3 Levelshift"
- note added: "Decoupling"
- note added: "Mic Array"
- note added: "PDM -> TDM Multiplexer"
- note added: "Sentinel Mic"

Commit message: Fixed footprints and some not connected caps
Parts:
- R23: renamed from R17; footprint PCM_JLCPCB:R_0402 -> Resistor_SMD:R_0402_1005Metric
- R24: renamed from R18; footprint PCM_JLCPCB:R_0402 -> Resistor_SMD:R_0402_1005Metric
- R25: renamed from R19; footprint PCM_JLCPCB:R_0402 -> Resistor_SMD:R_0402_1005Metric
- R26: renamed from R20; footprint PCM_JLCPCB:R_0402 -> Resistor_SMD:R_0402_1005Metric
- R27: renamed from R21; footprint PCM_JLCPCB:R_0402 -> Resistor_SMD:R_0402_1005Metric
- R28: renamed from R22; footprint PCM_JLCPCB:R_0402 -> Resistor_SMD:R_0402_1005Metric
- R29: renamed from R26; footprint PCM_JLCPCB:R_0402 -> Resistor_SMD:R_0402_1005Metric
- R30: renamed from R25; footprint PCM_JLCPCB:R_0402 -> Resistor_SMD:R_0402_1005Metric
- R31: renamed from R24; footprint PCM_JLCPCB:R_0402 -> Resistor_SMD:R_0402_1005Metric
- R32: renamed from R23; footprint PCM_JLCPCB:R_0402 -> Resistor_SMD:R_0402_1005Metric
- R33: renamed from R27; footprint PCM_JLCPCB:R_0402 -> Resistor_SMD:R_0402_1005Metric
- renumbered C31 to C28, C30 to C29, C33 to C30, C32 to C31, C29 to C32, C28 to C33, C35 to C34, C34 to C35
Connections:
- net 1V8: now also C30.1, C31.2

Commit message: Finished scem
Connections:
- net 1V8: no longer C17.1, C18.1, C19.1, C20.1, C21.1, C22.1, C23.1, C24.1, C25.1, C30.1, C31.2, MK1.7 (VDD), MK2.7 (VDD), MK3.7 (VDD), MK4.7 (VDD), MK5.7 (VDD), MK6.7 (VDD), MK7.5 (THSEL), U10.3 (A), U8.1 (AVDD)
- new net: MK7.5 (THSEL), U10.3 (A)
- new net 1V8_SW: C17.1, C18.1, C19.1, C20.1, C21.1, C22.1, C23.1, C24.1, C25.1, C30.1, C31.2, MK1.7 (VDD), MK2.7 (VDD), MK3.7 (VDD), MK4.7 (VDD), MK5.7 (VDD), MK6.7 (VDD), U8.1 (AVDD)
Changed lines of the file:
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@@
 	(text "PDM -> TDM Multiplexer\n"
 		(exclude_from_sim no)
-		(at 176.53 104.14 0)
+		(at 176.784 102.616 0)
 		(effects
 			(font
@@
 	)
 	(junction
-		(at 173.99 66.04)
-		(diameter 0)
-		(color 0 0 0 0)
-	)
-	(junction
 		(at 85.09 173.99)
 		(diameter 0)
@@
 	)
 	(junction
-		(at 182.88 66.04)
-		(diameter 0)
-		(color 0 0 0 0)
-	)
-	(junction
 		(at 83.82 90.17)
 		(diameter 0)
@@
 	(wire
 		(pts
-			(xy 173.99 66.04) (xy 182.88 66.04)
+			(xy 80.01 173.99) (xy 85.09 173.99)
 		)
 		(stroke
@@
 	(wire
 		(pts
-			(xy 80.01 173.99) (xy 85.09 173.99)
+			(xy 144.78 135.89) (xy 154.9398 135.89)
 		)
 		(stroke
@@
 	(wire
 		(pts
-			(xy 144.78 135.89) (xy 154.9398 135.89)
+			(xy 54.61 114.3) (xy 54.61 137.16)
 		)
 		(stroke
@@
 	(wire
 		(pts
-			(xy 54.61 114.3) (xy 54.61 137.16)
+			(xy 83.82 78.74) (xy 83.82 90.17)
 		)
 		(stroke
@@
 	(wire
 		(pts
-			(xy 83.82 78.74) (xy 83.82 90.17)
+			(xy 205.74 138.43) (xy 209.55 138.43)
 		)
 		(stroke
@@
 	(wire
 		(pts
-			(xy 205.74 138.43) (xy 209.55 138.43)
+			(xy 90.17 181.61) (xy 95.25 181.61)
 		)
 		(stroke
@@
 	(wire
 		(pts
-			(xy 90.17 181.61) (xy 95.25 181.61)
+			(xy 182.8801 110.49) (xy 182.88 111.76)
 		)
 		(stroke
@@
 	(wire
 		(pts
-			(xy 144.78 140.97) (xy 154.9398 140.97)
+			(xy 180.34 110.49) (xy 180.3399 111.76)
 		)
 		(stroke
@@
 	(wire
 		(pts
-			(xy 173.99 46.99) (xy 179.07 46.99)
+			(xy 144.78 140.97) (xy 154.9398 140.97)
 		)
 		(stroke
@@
 	(wire
 		(pts
-			(xy 173.99 66.04) (xy 173.99 76.2)
+			(xy 173.99 46.99) (xy 179.07 46.99)
 		)
 		(stroke
@@
 	(wire
 		(pts
-			(xy 173.99 53.34) (xy 173.99 66.04)
+			(xy 173.99 53.34) (xy 173.99 76.2)
 		)
 		(stroke
@@
 	(wire
 		(pts
-			(xy 180.3399 111.76) (xy 186.69 111.76)
+			(xy 180.34 110.49) (xy 182.8801 110.49)
 		)
 		(stroke
@@
 		(in_pos_files yes)
 		(dnp no)
-		(fields_autoplaced yes)
 		(property "Reference" "#PWR057"
 			(at 53.34 48.26 0)
@@
 			)
 		)
-		(property "Value" "1V8"
-			(at 53.34 40.005 0)
+		(property "Value" "1V8_SW"
+			(at 52.324 40.894 0)
 			(show_name no)
 			(do_not_autoplace no)
@@
 	(symbol
 		(lib_id "power:GND")
-		(at 186.69 111.76 0)
+		(at 182.88 111.76 0)
 		(unit 1)
 		(body_style 1)
@@
 		(fields_autoplaced yes)
 		(property "Reference" "#PWR078"
-			(at 186.69 118.11 0)
+			(at 182.88 118.11 0)
 			(hide yes)
 			(show_name no)
@@
 		)
 		(property "Value" "GND"
-			(at 186.69 116.84 0)
+			(at 182.88 116.84 0)
 			(hide yes)
 			(show_name no)
@@
 		)
 		(property "Footprint" ""
-			(at 186.69 111.76 0)
+			(at 182.88 111.76 0)
 			(hide yes)
 			(show_name no)
@@
 		)
 		(property "Datasheet" ""
-			(at 186.69 111.76 0)
+			(at 182.88 111.76 0)
 			(hide yes)
 			(show_name no)
@@
 		)
 		(property "Description" "Power symbol creates a global label with name \"GND\" , ground"
-			(at 186.69 111.76 0)
+			(at 182.88 111.76 0)
 			(hide yes)
 			(show_name no)
@@
 		(in_pos_files yes)
 		(dnp no)
-		(fields_autoplaced yes)
 		(property "Reference" "#PWR073"
 			(at 153.67 113.03 0)
@@
 			)
 		)
-		(property "Value" "1V8"
-			(at 153.67 104.775 0)
+		(property "Value" "1V8_SW"
+			(at 153.67 105.41 0)
 			(show_name no)
 			(do_not_autoplace no)

Commit message: Reanotated
Parts:
- renumbered C17 to C23, C18 to C24, C19 to C25, C20 to C26, C21 to C27, C22 to C28, C23 to C29, C24 to C30, C25 to C31, C26 to C32, C27 to C33, C28 to C34, C29 to C35, C30 to C36, C31 to C37, C32 to C38, C33 to C39, C34 to C40, C35 to C41, C36 to C42, C37 to C43, R23 to R29, R24 to R30, R25 to R31, R26 to R32, R27 to R33, R28 to R34, R29 to R35, R30 to R36, R31 to R37, R32 to R38, R33 to R39, U9 to U10, U10 to U11, U8 to U9

Commit message: Added Mics
Parts:
- U9: footprint Package_DFN_QFN:QFN-28_4x4mm_P0.5mm -> Package_DFN_QFN:WQFN-24-1EP_4x4mm_P0.5mm_EP2.45x2.45mm_ThermalVias
Changed lines of the file:
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@@
 			)
 		)
-		(property "Footprint" "Package_DFN_QFN:QFN-28_4x4mm_P0.5mm"
+		(property "Footprint" "Package_DFN_QFN:WQFN-24-1EP_4x4mm_P0.5mm_EP2.45x2.45mm_ThermalVias"
 			(at 180.3399 132.08 0)
 			(hide yes)

Commit message: lots of routing to be done
maybe its time to descope...
Parts:
- renumbered R29 to R28, R30 to R29, R31 to R30, R32 to R31, R33 to R32, R34 to R33, R35 to R34, R36 to R35, R37 to R36, R38 to R37, R39 to R38
Connections:
- net 1V8: no longer MK1.2 (SELECT), MK3.2 (SELECT), MK5.2 (SELECT)
- net 1V8_SW: now also MK1.2 (SELECT), MK3.2 (SELECT), MK5.2 (SELECT)

Commit message: Layout more or less done. Still missing i2c pullups and need to redo pinout
Parts:
- renumbered C23 to C24, C24 to C25, C25 to C26, C26 to C27, C27 to C28, C28 to C29, C29 to C30, C30 to C31, C31 to C32, C32 to C33, C33 to C34, C34 to C35, C35 to C36, C36 to C37, C37 to C38, C38 to C39, C39 to C40, C40 to C41, C41 to C42, C42 to C43, C43 to C44, R28 to R27, R29 to R28, R30 to R29, R31 to R30, R32 to R31, R33 to R32, R34 to R33, R35 to R34, R36 to R35, R37 to R36, R38 to R37
Connections:
- net 1V8: now also C30.1, C31.1, C32.1
- net 1V8_SW: no longer C30.1, C31.1, C32.1
Other:
- moved on the sheet: C30, C31, C32
